Commit message: Add files via upload

File: my_robot_description/urdf/mobile_base.xacro (robot description, xacro)
@@ -82,5 +82,5 @@
         <parent link="base_link" />
         <child link="caster_wheel_link" />
-        <origin xyz="${-base_length / 3.0} 0 ${-wheel_radius / 2.0}" rpy="0 0 0" />
+        <origin xyz="${base_length / 3.0} 0 ${-wheel_radius / 2.0}" rpy="0 0 0" />
     </joint>
 </robot>
